File: semi-controlled-rectifier-breakout-board.sch (EAGLE design)
At the start: 16 parts, among them U10 VO3053-X007T, U11 VO3053-X007T, U8 TN4015H-6G, U9 TN4015H-6G, X1 22-23-2031

Commit message: Modified flatcam files and brd layout
Connections:
- net P1_FUSED: no longer U11A.A2
- net P2_IN: now also U11A.A2
Changed lines of the file:
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@@
 <pinref part="U9" gate="A" pin="A"/>
 <wire x1="71.12" y1="5.08" x2="86.36" y2="5.08" width="0.1524" layer="91"/>
-<wire x1="86.36" y1="5.08" x2="104.14" y2="5.08" width="0.1524" layer="91"/>
+<wire x1="86.36" y1="5.08" x2="93.98" y2="5.08" width="0.1524" layer="91"/>
+<wire x1="93.98" y1="5.08" x2="104.14" y2="5.08" width="0.1524" layer="91"/>
 <wire x1="86.36" y1="5.08" x2="86.36" y2="-2.54" width="0.1524" layer="91"/>
 <junction x="86.36" y="5.08"/>
 <label x="86.36" y="-2.54" size="1.778" layer="95" rot="R270" xref="yes"/>
+<wire x1="175.26" y1="12.7" x2="175.26" y2="-17.78" width="0.1524" layer="91"/>
+<wire x1="175.26" y1="-17.78" x2="93.98" y2="-17.78" width="0.1524" layer="91"/>
+<wire x1="93.98" y1="-17.78" x2="93.98" y2="5.08" width="0.1524" layer="91"/>
+<junction x="93.98" y="5.08"/>
+<pinref part="U11" gate="A" pin="A2"/>
+<wire x1="175.26" y1="12.7" x2="167.64" y2="12.7" width="0.1524" layer="91"/>
 </segment>
 <segment>
@@
 <wire x1="86.36" y1="66.04" x2="172.72" y2="66.04" width="0.1524" layer="91"/>
 <junction x="86.36" y="66.04"/>
-<pinref part="U11" gate="A" pin="A2"/>
 <wire x1="172.72" y1="66.04" x2="172.72" y2="53.34" width="0.1524" layer="91"/>
-<wire x1="172.72" y1="53.34" x2="172.72" y2="12.7" width="0.1524" layer="91"/>
-<wire x1="172.72" y1="12.7" x2="167.64" y2="12.7" width="0.1524" layer="91"/>
 <pinref part="U10" gate="A" pin="A2"/>
 <wire x1="167.64" y1="53.34" x2="172.72" y2="53.34" width="0.1524" layer="91"/>
-<junction x="172.72" y="53.34"/>
 </segment>
 <segment>

Commit message: Created new cam file, started new flatcam project, and added silkscreen layer for labeling
Parts:
- added D1, D2: DIODE, RectifierParts:DIODE
- R20A, R20B: value (none) -> 200; device rcl:R-US_0207/7 -> RectifierParts:TH_RESISTOR
- R6A, R6B: value (none) -> 180; device rcl:R-US_0207/7 -> RectifierParts:TH_RESISTOR
Connections:
- new net N$3: D1.C, U11A.A2
- new net N$9: D2.C, U10A.A2
- net N$2: now also R6A.P$2; no longer R6A.2
- net N$4: now also R6B.P$2; no longer R6B.2
- net N$5: now also R6A.P$1; no longer R6A.1
- net N$6: now also R6B.P$1; no longer R6B.1
- net N$7: now also R20A.P$2; no longer R20A.2
- net N$8: now also R20B.P$2; no longer R20B.2
- net P1_FUSED: now also D2.A; no longer U10A.A2
- net P2_IN: now also D1.A; no longer U11A.A2
- net PHASE_CONTROL_SIGNAL: now also R20A.P$1, R20B.P$1; no longer R20A.1, R20B.1
